File: macropad/macropad.sch (KiCad schematic (older format))
At the start: 21 parts, among them J1 AVR_ISP_6, J2 Conn_01x04, J3 USB_OTG, SW1 RESET, SW2 BOOT, U1 ATmega328-PU, Y1 16MHz

Commit message: keebio kicad libs
Parts:
- added D? (x12): D_Small, symbol Device:D_Small
- added MX? (x12): MX-1U, symbol MX_Alps_Hybrids:MX-1U
